File: hw/Programmable battery power saving board.sch (KiCad schematic (older format))
At the start: 26 parts, among them P1 277-9143, P2 power_in, P3 power_out, Q1 TN0606N3-G, Q2 TN0606N3-G, Q3 TN0606N3-G, Q4 IPP45P03P4L-11, Q5 TN0606N3-G, Q6 LP0701N3-G, SW1 SW_PUSH, SW2 SW_PUSH, U11 DS3231S

Commit message: Last changed from Eloise
Parts:
- BT1: symbol Battery -> Battery-RESCUE-Programmable_battery_power_saving_board
Changed lines of the file:
@@
 EESchema Schematic File Version 2
+LIBS:Programmable battery power saving board-rescue
 LIBS:power
 LIBS:device
@@
 LIBS:contrib
 LIBS:valves
-LIBS:ds3231s
-LIBS:PowerManagementBoard-cache
+LIBS:Programmable battery power saving board-cache
 EELAYER 25 0
 EELAYER END
@@
 $EndComp
 $Comp
-L Battery BT1
+L Battery-RESCUE-Programmable_battery_power_saving_board BT1
 U 1 1 58938CBB
 P 7850 2400
